File: Tester_circut/Motor_drivers.kicad_sch (KiCad schematic)
At the start: 16 parts, among them J1 KF301-2P, J2 KF301-2P, J3 KF301-2P, J4 KF301-2P, J5 KF301-2P, J6 KF301-2P, J7 KF301-2P, J8 KF301-2P, U13 TMC2209_SILENTSTEPSTICK, U2 TMC2209_SILENTSTEPSTICK, U3 TMC2209_SILENTSTEPSTICK, U5 TMC2209_SILENTSTEPSTICK

Commit message: schematic update
probably final update
Connections:
- net USART2_RX: no longer R4.1, R5.1, R8.1, U2.12 (UART), U3.12 (UART), U5.12 (UART)
- net USART2_TX: no longer R4.2, R5.2, R8.2
- new net USART4_RX: R8.1, U2.12 (UART)
- new net USART4_TX: R8.2
- new net USART5_RX: R5.1, U3.12 (UART)
- new net USART5_TX: R5.2
- new net USART6_RX: R4.1, U5.12 (UART)
- new net USART6_TX: R4.2
