File: Tester_circut/Tester_circut.kicad_sch (KiCad schematic)
At the start: 8 parts, among them SW1 Encoder, SW2 SW_DPST_x2, U4 LCD, U9 Power_supply

Commit message: schematic update
probably final update
Connections:
- net EndStop1: now also A1.CN10_2 (D7/IO); no longer A1.CN10_10 (D3/TIMER_A_PWM3)
- net Test_pin: now also A1.CN10_10 (D3/TIMER_A_PWM3); no longer A1.CN9_1 (A0/ADC123_IN3)
- net diag1: now also A1.CN10_16 (D0/USART_A_RX)
- net diag2: now also A1.CN10_15 (D27/QSPI_CLK)
- net diag3: now also A1.CN10_13 (D26/QSPI_CS)
- net diag4: now also A1.CN10_11 (A8/ADC_C_IN)
- net USART5_TX: now reaches A1.CN8_10 (D47/SDMMC_CK)
- net USART5_RX: now reaches A1.CN8_12 (D48/SDMMC_CMD)
- net USART4_TX: now reaches A1.CN8_6 (D45/SDMMC_D2)
- net USART4_RX: now reaches A1.CN8_8 (D46/SDMMC_D3)
- net USART6_TX: now reaches A1.CN7_1 (D16/I2S_A_MCK)
- net USART6_RX: now reaches A1.CN7_11 (D21/I2S_B_MCK)
- no-connect marks 53 -> 44
Other:
- sheet End stop sensors ports: added none; removed +5V
- sheet Motor drivers ports: added USART4_RX, USART4_TX, USART5_RX, USART5_TX, USART6_RX, USART6_TX; removed none
- moved on the sheet: A1C, A1F
